File: hardware/SoilMoistureSensor.kicad_sch (KiCad schematic)
At the start: 36 parts, among them J1 Conn_01x02, J2 Conn_01x04, J3 Conn_01x02, Q1 AO3401A, SW1 SW_Push, SW2 SW_Push, U1 BQ25570, U2 ESP32-C3-WROOM-02, U3 TLC555xD

Commit message: created schematic and pcb
Other:
- note added: "PF1-PF5: ERC power-source markers for nets fed by an external/passive element ERC cannot verify (solar panel, supercap, regulated rail, load-switched rail) - not real parts."
- note removed: "PF1-PF4: ERC power-source markers for nets fed by an external/passive element ERC cannot verify (solar panel, supercap, regulated rail, load-switched rail) - not real parts."

Commit message: completed routing of board. still need to add capacitive sensing traces
Parts:
- J1, J3: footprint (none) -> Connector_JST:JST_PH_B2B-PH-K_1x02_P2.00mm_Vertical
- J2: footprint (none) -> Connector_PinHeader_2.54mm:PinHeader_1x04_P2.54mm_Vertical
- L1, L2: footprint (none) -> Inductor_SMD:L_APV_ANR4030
- SC1: footprint (none) -> Capacitor_THT:CP_Radial_D13.0mm_P5.00mm
Changed lines of the file:
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@@
 			)
 		)
-		(property "Footprint" ""
+		(property "Footprint" "Capacitor_THT:CP_Radial_D13.0mm_P5.00mm"
 			(at 90.17 165.1 0)
 			(hide yes)
@@
 			)
 		)
-		(property "Footprint" ""
+		(property "Footprint" "Inductor_SMD:L_APV_ANR4030"
 			(at 90.17 39.37 0)
 			(hide yes)
@@
 			)
 		)
-		(property "Footprint" ""
+		(property "Footprint" "Connector_PinHeader_2.54mm:PinHeader_1x04_P2.54mm_Vertical"
 			(at 444.5 149.86 0)
 			(hide yes)
@@
 			)
 		)
-		(property "Footprint" ""
+		(property "Footprint" "Connector_JST:JST_PH_B2B-PH-K_1x02_P2.00mm_Vertical"
 			(at 30.48 59.69 0)
 			(hide yes)
@@
 			)
 		)
-		(property "Footprint" ""
+		(property "Footprint" "Inductor_SMD:L_APV_ANR4030"
 			(at 229.87 59.69 0)
 			(hide yes)
@@
 			)
 		)
-		(property "Footprint" ""
+		(property "Footprint" "Connector_JST:JST_PH_B2B-PH-K_1x02_P2.00mm_Vertical"
 			(at 459.74 260.35 0)
 			(hide yes)

Commit message: astra redesigned then ran out of usage
Parts:
- removed C1: 4.7uF, Capacitor_SMD:C_1206_3216Metric, symbol Device:C
- removed C11, C5, C8, C9: 100nF, Capacitor_SMD:C_0805_2012Metric, symbol Device:C
- removed C2: 4.7uF, Capacitor_SMD:C_0805_2012Metric, symbol Device:C
- removed C3: 0.1uF, Capacitor_SMD:C_0805_2012Metric, symbol Device:C
- removed C4: 10nF, Capacitor_SMD:C_0805_2012Metric, symbol Device:C
- removed C6: 22uF, Capacitor_SMD:C_1206_3216Metric, symbol Device:C
- removed C7: 10uF, Capacitor_SMD:C_0805_2012Metric, symbol Device:C
- removed J1, J3: Conn_01x02, Connector_JST:JST_PH_B2B-PH-K_1x02_P2.00mm_Vertical, symbol Connector_Generic:Conn_01x02
- removed J2: Conn_01x04, Connector_PinHeader_2.54mm:PinHeader_1x04_P2.54mm_Vertical, symbol Connector_Generic:Conn_01x04
- removed L1: 22uH, Inductor_SMD:L_APV_ANR4030, symbol Device:L
- removed L2: 10uH, Inductor_SMD:L_APV_ANR4030, symbol Device:L
- removed Q1: AO3401A, Package_TO_SOT_SMD:SOT-23, symbol Transistor_FET:AO3401A
- removed R1: 3.01M 1%, Resistor_SMD:R_0805_2012Metric, symbol Device:R
- removed R10, R12: 1k, Resistor_SMD:R_0805_2012Metric, symbol Device:R
- removed R11: 100k, Resistor_SMD:R_0805_2012Metric, symbol Device:R
- removed R13: 4.7k, Resistor_SMD:R_0805_2012Metric, symbol Device:R
- removed R2: 10.0M 1%, Resistor_SMD:R_0805_2012Metric, symbol Device:R
- removed R3: 2.49M 1%, Resistor_SMD:R_0805_2012Metric, symbol Device:R
- removed R4: 4.99M 1%, Resistor_SMD:R_0805_2012Metric, symbol Device:R
- removed R5: 866k 1%, Resistor_SMD:R_0805_2012Metric, symbol Device:R
- removed R6: 4.75M 1%, Resistor_SMD:R_0805_2012Metric, symbol Device:R
- removed R7: 8.25M 1%, Resistor_SMD:R_0805_2012Metric, symbol Device:R
- removed R8, R9: 10k, Resistor_SMD:R_0805_2012Metric, symbol Device:R
- removed RV1: 10k trim, Potentiometer_THT:Potentiometer_Bourns_3296W_Vertical, symbol Device:R_Potentiometer_Trim
- removed SC1: 3F 5.5V Supercap, Capacitor_THT:CP_Radial_D13.0mm_P5.00mm, symbol Device:C_Polarized
- removed SW1, SW2: SW_Push, Button_Switch_SMD:SW_SPST_TL3342, symbol Switch:SW_Push
- removed U1: BQ25570, Package_DFN_QFN:QFN-20-1EP_3.5x3.5mm_P0.5mm_EP2x2mm, symbol Battery_Management:BQ25570
- removed U2: ESP32-C3-WROOM-02, RF_Module:ESP32-C3-WROOM-02, symbol RF_Module:ESP32-C3-WROOM-02
- removed U3: TLC555xD, Package_SO:SOIC-8_3.9x4.9mm_P1.27mm, symbol Timer:TLC555xD
- added C1: 4.7uF 10V X7R, Capacitor_SMD:C_1206_3216Metric, symbol MoistureRevB:C
- added C10, C3, C5, C8, C9: 100nF 10V, Capacitor_SMD:C_0805_2012Metric, symbol MoistureRevB:C
- added C11: 10nF, Capacitor_SMD:C_0805_2012Metric, symbol MoistureRevB:C
- added C12, C7: 10uF 10V X7R, Capacitor_SMD:C_0805_2012Metric, symbol MoistureRevB:C
- added C2: 4.7uF 10V X7R, Capacitor_SMD:C_0805_2012Metric, symbol MoistureRevB:C
- added C4: 10nF C0G 5%, Capacitor_SMD:C_0805_2012Metric, symbol MoistureRevB:C
- added C6: 10uF 10V X7R, Capacitor_SMD:C_1206_3216Metric, symbol MoistureRevB:C
- added J1, J3: Conn_01x02, Connector_JST:JST_PH_B2B-PH-K_1x02_P2.00mm_Vertical, symbol MoistureRevB:Conn_01x02
- added J2: Conn_01x04, Connector_PinHeader_2.54mm:PinHeader_1x04_P2.54mm_Vertical, symbol MoistureRevB:Conn_01x04
- added J4: PCB capacitive probe, SoilProbe:SoilProbe_IDC_40x30mm, symbol MoistureRevB:Conn_01x02
- added L1: 22uH / Isat >= 0.4A, Inductor_SMD:L_Coilcraft_LPS4018, symbol MoistureRevB:L
- added L2: 2.2uH / Isat >= 1.5A, Inductor_SMD:L_Coilcraft_LPS4018, symbol MoistureRevB:L
- added Q1: AO3401A, Package_TO_SOT_SMD:SOT-23, symbol MoistureRevB:AO3401A
- added R1: 4.75M 1%, Resistor_SMD:R_0805_2012Metric, symbol MoistureRevB:R
- added R10: 1k, Resistor_SMD:R_0805_2012Metric, symbol MoistureRevB:R
- added R11: 100k, Resistor_SMD:R_0805_2012Metric, symbol MoistureRevB:R
- added R12, R14, R15, R8, R9: 10k, Resistor_SMD:R_0805_2012Metric, symbol MoistureRevB:R
- added R13: 47k, Resistor_SMD:R_0805_2012Metric, symbol MoistureRevB:R
- added R16: 52.3k 1%, Resistor_SMD:R_0805_2012Metric, symbol MoistureRevB:R
- added R2: 8.25M 1%, Resistor_SMD:R_0805_2012Metric, symbol MoistureRevB:R
- added R3: 2.49M 1%, Resistor_SMD:R_0805_2012Metric, symbol MoistureRevB:R
- added R4: 4.99M 1%, Resistor_SMD:R_0805_2012Metric, symbol MoistureRevB:R
- added R5: 866k 1%, Resistor_SMD:R_0805_2012Metric, symbol MoistureRevB:R
- added RV1: 100k trim, Potentiometer_THT:Potentiometer_Bourns_3296W_Vertical, symbol MoistureRevB:R_Potentiometer_Trim
- added SC1: 3F 5.4V PHV-5R4V305-R, SoilProbe:CP_Eaton_PHV_3F_Vertical_P11.8mm, symbol MoistureRevB:C_Polarized
- added SW1, SW2: SW_Push, Button_Switch_SMD:SW_SPST_TL3342, symbol MoistureRevB:SW_Push
- added U1: BQ25570, Package_DFN_QFN:QFN-20-1EP_3.5x3.5mm_P0.5mm_EP2x2mm, symbol MoistureRevB:BQ25570
- added U2: ESP32-C3-WROOM-02, RF_Module:ESP32-C3-WROOM-02, symbol MoistureRevB:ESP32-C3-WROOM-02
- added U3: TLC555xD, Package_SO:SOIC-8_3.9x4.9mm_P1.27mm, symbol MoistureRevB:TLC555xD
- added U4: TPS62842DGRR, Package_SO:HVSSOP-8-1EP_3x3mm_P0.65mm_EP1.57x1.89mm, symbol MoistureRevB:TPS62842DGR
Connections:
- net +3V3: now also C6.1, C7.1, C8.1, J2.1 (Pin_1), L2.2, Q1.2 (S), R11.1, R14.1, R15.1, R8.1, R9.1, U2.1 (3V3), U4.1 (VOS)
- net BAT_OK: now also U1.13 (VBAT_OK), U4.5 (EN)
- net CTRL_BP: now also C11.1, U3.5 (CONT)
- net EN_ESP: now also C9.1, R8.2, SW1.1, U2.2 (EN)
- net ESP_RXD: now also J2.4 (Pin_4), U2.11 (IO20/RXD)
- net ESP_TXD: now also J2.3 (Pin_3), U2.12 (IO21/TXD)
- net FREQ_IN: now also U2.4 (IO5), U3.3 (OUT)
- net GND: now also C1.2, C10.2, C11.2, C12.2, C2.2, C3.2, C4.2, C5.2, C6.2, C7.2, C8.2, C9.2, J1.2 (Pin_2), J2.2 (Pin_2), J3.2 (Pin_2), J4.2 (Pin_2), R1.2, R16.2, R3.1, SC1.2, SW1.2, SW2.2, U1.1 (VSS), U1.12 (VOUT_SET), U1.15 (VSS), U1.17 (VSS), U1.21 (VSS), U1.5 (~{EN}), U1.6 (VOUT_EN), U1.9 (VSS), U2.19 (GND), U2.9 (GND), U3.1 (GND), U4.3 (MODE), U4.8 (GND), U4.9 (EP)
- net GPIO9_BOOT: now also R9.2, SW2.1, U2.8 (IO9)
- net LBOOST: now also L1.2, U1.20 (LBOOST)
- net OK_HYST_N: now also R4.2, R5.2, U1.10 (OK_HYST)
- net OK_PROG_N: now also R3.2, R4.1, U1.11 (OK_PROG)
- net OSC_RC: now also J3.1 (Pin_1), J4.1 (Pin_1), RV1.3, U3.2 (TRIG), U3.6 (THRES)
- net OSC_RC_DISCH: now also R12.2, R13.1, U3.7 (DISCH)
- net RV1_WIPER_TIE: now also R13.2, RV1.1, RV1.2
- net SENSOR_GATE: now also Q1.1 (G), R10.2, R11.2
- net SENSOR_PWR_EN: now also R10.1, U2.3 (IO4)
- net VBAT: now also C12.1, C5.1, SC1.1, U1.18 (VBAT), U4.6 (VIN)
- net VBAT_OV_N: now also R1.1, R2.2, U1.7 (VBAT_OV)
- net VCC_SENSOR: now also C10.1, Q1.3 (D), R12.1, U3.4 (~{RST}), U3.8 (VCC)
- net VIN_DC: now also C1.1, J1.1 (Pin_1), L1.1, U1.2 (VIN_DC)
- net VRDIV: now also R2.1, R5.1, U1.8 (VRDIV)
- net VREF_SAMP: now also C4.1, U1.4 (VREF_SAMP)
- net VSTOR: now also C2.1, C3.1, U1.19 (VSTOR), U1.3 (VOC_SAMP)
- new net BUCK_SW: L2.1, U4.2 (SW)
- new net BUCK_VSET: R16.1, U4.4 (VSET)
- new net GPIO2_BOOT: R15.2, U2.16 (IO2)
- new net GPIO8_BOOT: R14.2, U2.7 (IO8)
- no-connect marks 10 -> 11
Other:
- note added: "01 ENERGY HARVESTING + STORAGE"
- note added: "02 ESP32-C3 + PROGRAMMING"
- note added: "03 3.3 V / 750 mA SUPPLY"
- note added: "04 SWITCHED CAPACITIVE OSCILLATOR"
- note added: "BQ25570 buck disabled. VOUT/LBUCK intentionally open. U4 draws from VBAT directly; BAT_OK provides hysteretic shutdown. R1/R2: OV = 1.5 x 1.21 x (1 + 8.25/4.75) = 4.967 V. R3/R4/R5: OFF 3.635 V; ON 4.056 V. J1: solar source only; Voc <= 5.1 V and power <= 400 mW. SC1: Eaton PHV-5R4V305-R, low ESR. Indoor use, <= 65 C."
- note added: "GPIO4 LOW = sensor ON; HIGH = OFF. Retain HIGH in sleep. Measure frequency on GPIO5 after sensor settling; radio off during measurement. J3 is an optional external probe/test connector, parallel with J4. J4 copper is covered by solder mask. Seal probe edges before soil exposure. Calibrate dry/wet in the actual soil and coating; frequency is not absolute VWC. J2 pin 1 is 3.3 V OUTPUT/reference, no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"
- note added: "POWER-NET ERC FLAGS (passive storage / switched power)"
- note removed: "BQ25570 programming (see datasheet SLUSBH2G eqs 1-5): R1/R2 -> VBAT_OV ~5.23V (supercap overvoltage cutoff) R3/R4/R5 -> VBAT_OK falls 3.64V / rises 4.06V (auto load gate) R6/R7 -> VOUT ~3.31V regulated system rail VOC_SAMP tied to VSTOR = 80% MPPT for solar"
- note removed: "CAPACITIVE PROBE OSCILLATOR (power-gated by MCU)"
- note removed: "ESP32-C3 MCU / UART PROGRAMMING HEADER"
- note removed: "J2: UART programming header 1=3V3 2=GND 3=ESP TXD 4=ESP RXD (external USB-serial adapter: adapter RX->pin3, adapter TX->pin4)"
- note removed: "J3: capacitive probe plates (placeholder - real "connector" is a copper-pour comb pattern laid out on the PCB itself, not an off-board connector). RA=R12, RB=R13+RV1 (trim pot) - tune once probe C is characterized; use ESP32-C3 PCNT peripheral to count FREQ_IN edges."
- note removed: "PF1-PF5: ERC power-source markers for nets fed by an external/passive element ERC cannot verify (solar panel, supercap, regulated rail, load-switched rail) - not real parts."
- note removed: "SC1: single-cell supercapacitor, >=100uF equiv, 5.5V rated. Footprint per chosen part."
- note removed: "SOLAR ENERGY HARVESTER / SUPERCAP STORAGE / 3V3 SYSTEM RAIL"
- note removed: "SOLAR PANEL (small indoor PV, ~5.5V Voc)"
- note removed: "SW1: reset (EN)"
- note removed: "SW2: boot (hold, then tap reset)"
- title: Soil Moisture Sensor Module -> Soil moisture sensor - solar / supercapacitor
