File: hardware/SoilMoistureSensor.kicad_sch (KiCad schematic)
At the start: 48 parts, among them J1 Conn_01x02, J2 Conn_01x04, J3 Conn_01x02, J4 PCB capacitive probe, Q1 AO3401A, SW1 TS-1088-AR02016, SW2 TS-1088-AR02016, U1 BQ25570, U2 ESP32-C3-WROOM-02-N4, U3 TLC555CDR, U4 TPS62842DGRR

Commit message: had claude go in and fix what astra didnt finish. extended length to 3.5inch
Parts:
- J4: footprint SoilProbe:SoilProbe_IDC_40x55mm -> SoilProbe:SoilProbe_IDC_40x85mm; now left out of the parts list
Changed lines of the file:
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@@
 		(at 541.02 281.94 0)
 		(unit 1)
-		(in_bom yes)
+		(in_bom no)
 		(on_board yes)
 		(dnp no)
@@
 			)
 		)
-		(property "Footprint" "SoilProbe:SoilProbe_IDC_40x55mm"
+		(property "Footprint" "SoilProbe:SoilProbe_IDC_40x85mm"
 			(at 541.02 281.94 0)
 			(effects
