File: review/revB/pre-extension.kicad_sch (KiCad schematic)
At the start: 48 parts, among them J1 Conn_01x02, J2 Conn_01x04, J3 Conn_01x02, J4 PCB capacitive probe, Q1 AO3401A, SW1 TS-1088-AR02016, SW2 TS-1088-AR02016, U1 BQ25570, U2 ESP32-C3-WROOM-02-N4, U3 TLC555CDR, U4 TPS62842DGRR

Commit message: told astra to lengthen board, choose solar panel, and keep all parts jlcpcb basic
Parts:
- removed R17, R18, R20, R21, R22, R23: 2M 1%, Resistor_SMD:R_0603_1608Metric, symbol MoistureRevB:R
- removed R19: 3M 1%, Resistor_SMD:R_0603_1608Metric, symbol MoistureRevB:R
- C1: value 4.7uF 25V X5R -> 4.7uF 10V X7R; footprint Capacitor_SMD:C_0805_2012Metric -> Capacitor_SMD:C_1206_3216Metric
- C10, C3, C5, C8, C9: value 100nF 50V X7R -> 100nF 10V
- C11: value 10nF 50V X7R -> 10nF
- C12, C7: value 10uF 25V X5R -> 10uF 10V X7R
- C2: value 4.7uF 25V X5R -> 4.7uF 10V X7R
- C6: value 10uF 25V X5R -> 10uF 10V X7R; footprint Capacitor_SMD:C_0805_2012Metric -> Capacitor_SMD:C_1206_3216Metric
- J1, J2, J3, RV1, SC1: now fitted
- J4: footprint SoilProbe:SoilProbe_IDC_40x55mm -> SoilProbe:SoilProbe_IDC_40x30mm
- R1: value 2M 1% -> 4.75M 1%; footprint Resistor_SMD:R_0603_1608Metric -> Resistor_SMD:R_0805_2012Metric
- R2: value 2M 1% -> 8.25M 1%; footprint Resistor_SMD:R_0603_1608Metric -> Resistor_SMD:R_0805_2012Metric
- R3: value 2M 1% -> 2.49M 1%; footprint Resistor_SMD:R_0603_1608Metric -> Resistor_SMD:R_0805_2012Metric
- R4: value 2M 1% -> 4.99M 1%; footprint Resistor_SMD:R_0603_1608Metric -> Resistor_SMD:R_0805_2012Metric
- R5: value 1.5M 1% -> 866k 1%; footprint Resistor_SMD:R_0603_1608Metric -> Resistor_SMD:R_0805_2012Metric
- SW1, SW2: value TS-1088-AR02016 -> SW_Push; footprint Button_Switch_SMD:SW_SPST_TS-1088-xR020 -> Button_Switch_SMD:SW_SPST_TL3342
- U2: value ESP32-C3-WROOM-02-N4 -> ESP32-C3-WROOM-02; footprint SoilProbe:ESP32-C3-WROOM-02_0.3mm_thermal_vias -> RF_Module:ESP32-C3-WROOM-02
- U3: value TLC555CDR -> TLC555xD
Connections:
- net OK_LO_SER is gone; now on net OK_PROG_N: R3.2
- net OK_MID_SER1 is gone; now on net OK_HYST_N: R4.2
- net OV_HI_SER1 is gone; now on net VBAT_OV_N: R2.2
- net OV_LO_SER is gone; now on net GND: R1.2
Other:
- note added: "BQ25570 buck disabled. VOUT/LBUCK intentionally open. U4 draws from VBAT directly; BAT_OK provides hysteretic shutdown. R1/R2: OV = 1.5 x 1.21 x (1 + 8.25/4.75) = 4.967 V. R3/R4/R5: OFF 3.635 V; ON 4.056 V. J1: solar source only; Voc <= 5.1 V and power <= 400 mW. SC1: Eaton PHV-5R4V305-R, low ESR. Indoor use, <= 65 C."
- note removed: "BQ25570 buck disabled; U4 draws from VBAT directly. OV: R1+R17 = 4M; R2+R18+R19 = 7M. OV = 1.5 x 1.21 x (1 + 7/4) = 4.991 V. BAT_OK: bottom 4M, middle 8M, top 1.5M. OFF = 3.630 V; ON = 4.084 V. Total divider = 13.5M. J1: solar Voc <= 5.1 V, power <= 400 mW. SC1: PHV-5R4V305-R, low ESR, indoor <= 65 C."
- moved on the sheet: R5
