File: review/before-inductor-swap/SoilMoistureSensor.kicad_pcb (KiCad board)
At the start: 2 copper layers, 55 x 198.5 mm, 55 parts, among them J1 Conn_01x02, J2 Conn_01x04, J3 Conn_01x02, J4 PCB capacitive probe, Q1 AO3401A, SW1 TS-1088-AR02016, SW2 TS-1088-AR02016, U1 BQ25570, U2 ESP32-C3-WROOM-02-N4, U3 TLC555CDR, U4 TPS62842DGRR

Commit message: reworked some parts to get jlcpcb basic, reworked inductors
Parts:
- L1, L2: footprint Inductor_SMD:L_Changjiang_FNR4018S -> Inductor_SMD:L_Coilcraft_LPS4018
Routing:
- net /LBOOST: track 4.13 -> 3.61 mm
