File: review/before-inductor-swap/SoilMoistureSensor.kicad_sch (KiCad schematic)
At the start: 51 parts, among them J1 Conn_01x02, J2 Conn_01x04, J3 Conn_01x02, J4 PCB capacitive probe, Q1 AO3401A, SW1 TS-1088-AR02016, SW2 TS-1088-AR02016, U1 BQ25570, U2 ESP32-C3-WROOM-02-N4, U3 TLC555CDR, U4 TPS62842DGRR

Commit message: reworked some parts to get jlcpcb basic, reworked inductors
Parts:
- L1: footprint Inductor_SMD:L_Changjiang_FNR4018S -> Inductor_SMD:L_Coilcraft_LPS4018; LCSC C167883 -> C5278935; MPN FNR4030S220MT -> LPS4018-223MRC; Manufacturer Changjiang Microelectronics -> Coilcraft; Source https://www.lcsc.com/product-detail/C167883.html -> https://www.lcsc.com/product-detail/C5278935.html
- L2: footprint Inductor_SMD:L_Changjiang_FNR4018S -> Inductor_SMD:L_Coilcraft_LPS4018; LCSC C167804 -> C4354938; MPN FNR4018S2R2MT -> LPS4018-222MRC; Manufacturer Changjiang Microelectronics -> Coilcraft; Source https://www.lcsc.com/product-detail/C167804.html -> https://www.lcsc.com/product-detail/C4354938.html
Changed lines of the file:
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@@
 			)
 		)
-		(property "Footprint" "Inductor_SMD:L_Changjiang_FNR4018S"
+		(property "Footprint" "Inductor_SMD:L_Coilcraft_LPS4018"
 			(at 42.1 81.28 0)
 			(effects
@@
 			)
 		)
-		(property "Manufacturer" "Changjiang Microelectronics"
+		(property "Manufacturer" "Coilcraft"
 			(at 38.1 81.28 0)
 			(effects
@@
 			)
 		)
-		(property "MPN" "FNR4030S220MT"
+		(property "MPN" "LPS4018-223MRC"
 			(at 38.1 81.28 0)
 			(effects
@@
 			)
 		)
-		(property "LCSC" "C167883"
+		(property "LCSC" "C5278935"
 			(at 38.1 81.28 0)
 			(effects
@@
 			)
 		)
-		(property "Source" "https://www.lcsc.com/product-detail/C167883.html"
+		(property "Source" "https://www.lcsc.com/product-detail/C5278935.html"
 			(at 38.1 81.28 0)
 			(effects
@@
 			)
 		)
-		(property "Footprint" "Inductor_SMD:L_Changjiang_FNR4018S"
+		(property "Footprint" "Inductor_SMD:L_Coilcraft_LPS4018"
 			(at 181.8 205.74 0)
 			(effects
@@
 			)
 		)
-		(property "Manufacturer" "Changjiang Microelectronics"
+		(property "Manufacturer" "Coilcraft"
 			(at 177.8 205.74 0)
 			(effects
@@
 			)
 		)
-		(property "MPN" "FNR4018S2R2MT"
+		(property "MPN" "LPS4018-222MRC"
 			(at 177.8 205.74 0)
 			(effects
@@
 			)
 		)
-		(property "LCSC" "C167804"
+		(property "LCSC" "C4354938"
 			(at 177.8 205.74 0)
 			(effects
@@
 			)
 		)
-		(property "Source" "https://www.lcsc.com/product-detail/C167804.html"
+		(property "Source" "https://www.lcsc.com/product-detail/C4354938.html"
 			(at 177.8 205.74 0)
 			(effects
