File: manufacture/source/SoilMoistureSensor.kicad_pcb (KiCad board)
At the start: 2 copper layers, 55 x 198.5 mm, 55 parts, among them J1 Conn_01x02, J2 Conn_01x04, J3 Conn_01x02, J4 PCB capacitive probe, Q1 AO3401A, SW1 TS-1088-AR02016, SW2 TS-1088-AR02016, U1 BQ25570, U2 ESP32-C3-WROOM-02-N4, U3 TLC555CDR, U4 TPS62842DGRR

Commit message: more fixes
Routing:
- net /+3V3: track 123.1 -> 139.4 mm
- net /OSC_RC_DISCH: track 16.3 -> 23.2 mm
- net /VRDIV: track 36.0 -> 42.1 mm
- net /OK_MID_SER1: track 5.25 -> 8.04 mm
- net /GPIO8_BOOT: track 19.1 -> 21.7 mm
- net /VBAT: track 107.4 -> 109.7 mm
- net /BAT_OK: track 19.0 -> 20.9 mm
- net /VIN_DC: track 53.2 -> 55.1 mm
